File: Electronics/590_Light_Project/initial_schematic.brd (EAGLE design)
At the start: 82.5 x 63.2 mm, 8 parts, among them U1 ARDUINOR3-DIMENSION

Commit message: Modified dimensions
Other:
- board size 82.5 x 63.2 mm -> 76.2 x 59.4 mm
Changed lines of the file:
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@@
 <board>
 <plain>
-<wire x1="30.48" y1="10.16" x2="113.01" y2="10.16" width="0" layer="20"/>
-<wire x1="113.01" y1="10.16" x2="113.01" y2="73.33" width="0" layer="20"/>
-<wire x1="113.01" y1="73.33" x2="30.48" y2="73.33" width="0" layer="20"/>
-<wire x1="30.48" y1="73.33" x2="30.48" y2="10.16" width="0" layer="20"/>
+<wire x1="34.29" y1="11.43" x2="110.47" y2="11.43" width="0" layer="20"/>
+<wire x1="110.47" y1="11.43" x2="110.47" y2="70.79" width="0" layer="20"/>
+<wire x1="110.47" y1="70.79" x2="34.29" y2="70.79" width="0" layer="20"/>
+<wire x1="34.29" y1="70.79" x2="34.29" y2="11.43" width="0" layer="20"/>
+<dimension x1="34.29" y1="11.43" x2="110.47" y2="11.43" x3="72.38" y3="8.89" textsize="1.778" layer="1"/>
+<dimension x1="101.6" y1="13.97" x2="101.6" y2="11.43" x3="115.57" y3="12.7" textsize="1.778" layer="1"/>
+<dimension x1="34.29" y1="70.79" x2="34.29" y2="11.43" x3="29.21" y3="41.11" textsize="1.778" layer="1"/>
+<dimension x1="38.1" y1="60.96" x2="34.29" y2="60.96" x3="36.195" y3="60.96" textsize="1.778" layer="1"/>
 </plain>
 <attributes>
